Commit message: description: set Yellow color to camera bounding box
Signed-off-by: Jean Laneurit <jean.laneurit@inrae.fr>

File: romea_stereo_camera_description/urdf/stereo_camera.xacro (robot description, xacro)
@@ -97,4 +97,5 @@
         <link name="${right_camera_optical_frame_name}"/>
         <gazebo reference="${link_name}">
+          <material>Gazebo/DarkYellow </material>
           <sensor type="multicamera" name="${prefix}${name}">
             <update_rate>${frame_rate}</update_rate>
@@ -166,4 +167,5 @@
                 </ros>
                 <camera_name>camera</camera_name>
+                <frame_name>${link_name}</frame_name>
             </plugin>
           </sensor>

Commit message: description: add simulation xacro file
Signed-off-by: Jean Laneurit <jean.laneurit@inrae.fr>

File: romea_stereo_camera_description/urdf/stereo_camera.xacro (robot description, xacro)
@@ -4,31 +4,49 @@
       params="prefix mode name configuration geometry xyz rpy parent_link mesh_visual ros_namespace">
         <xacro:property name="M_PI" value="3.1415926535897931" />
-        <xacro:property name="link_name" value="${prefix}${name}_link"/>
-        <xacro:property name="joint_name" value="${prefix}${name}_joint"/>
-        <xacro:property name="left_camera_link_name" value="${prefix}${name}_left_camera_link"/>
-        <xacro:property name="left_camera_joint_name" value="${prefix}${name}_left_camera_joint"/>
-        <xacro:property name="left_camera_optical_frame_name" value="${prefix}${name}_left_camera_optical_frame"/>
-        <xacro:property name="left_camera_optical_joint_name" value="${prefix}${name}_left_camera_optical_joint"/>
-        <xacro:property name="right_camera_link_name" value="${prefix}${name}_right_camera_link"/>
-        <xacro:property name="right_camera_joint_name" value="${prefix}${name}_right_camera_joint"/>
-        <xacro:property name="right_camera_optical_frame_name" value="${prefix}${name}_right_camera_optical_frame"/>
-        <xacro:property name="right_camera_optical_joint_name" value="${prefix}${name}_right_camera_optical_joint"/>
-        <xacro:property name="parent_link_name" value="${prefix}${parent_link}"/>
-        <xacro:property name="image_width" value="${configuration['image_width']}" />
-        <xacro:property name="image_height" value="${configuration['image_height']}" />
-        <xacro:property name="horizontal_fov" value="${configuration['horizontal_fov']}" />
-        <xacro:property name="frame_rate" value="${configuration['frame_rate']}" />
-        <xacro:property name="baseline" value="${geometry['baseline']}" />
-        <xacro:property name="mass" value="${geometry['mass']}" />
-        <xacro:property name="aabb" value="${geometry['aabb']}" />
-        <xacro:property name="aabb_length" value="${geometry['aabb']['length']}" />
-        <xacro:property name="aabb_width" value="${geometry['aabb']['width']}" />
-        <xacro:property name="aabb_height" value="${geometry['aabb']['height']}" />
-        <xacro:property name="aabb_center" value="${geometry['aabb']['center']}" />
+        <xacro:property name="link_name"
+          value="${prefix}${name}_link"/>
+        <xacro:property name="joint_name"
+          value="${prefix}${name}_joint"/>
+        <xacro:property name="left_camera_link_name"
+          value="${prefix}${name}_left_camera_link"/>
+        <xacro:property name="left_camera_joint_name"
+          value="${prefix}${name}_left_camera_joint"/>
+        <xacro:property name="left_camera_optical_frame_name"
+          value="${prefix}${name}_left_camera_optical_frame"/>
+        <xacro:property name="left_camera_optical_joint_name"
+          value="${prefix}${name}_left_camera_optical_joint"/>
+        <xacro:property name="right_camera_link_name"
+          value="${prefix}${name}_right_camera_link"/>
+        <xacro:property name="right_camera_joint_name"
+          value="${prefix}${name}_right_camera_joint"/>
+        <xacro:property name="right_camera_optical_frame_name"
+          value="${prefix}${name}_right_camera_optical_frame"/>
+        <xacro:property name="right_camera_optical_joint_name"
+          value="${prefix}${name}_right_camera_optical_joint"/>
+        <xacro:property name="parent_link_name"
+          value="${prefix}${parent_link}"/>
+        <xacro:property name="baseline"
+          value="${geometry['baseline']}" />
+        <xacro:property name="mass"
+          value="${geometry['mass']}" />
+        <xacro:property name="aabb"
+          value="${geometry['aabb']}" />
+        <xacro:property name="aabb_length"
+          value="${geometry['aabb']['length']}" />
+        <xacro:property name="aabb_width"
+          value="${geometry['aabb']['width']}" />
+        <xacro:property name="aabb_height"
+          value="${geometry['aabb']['height']}" />
+        <xacro:property name="aabb_center"
+          value="${geometry['aabb']['center']}" />
         <xacro:if value="${mesh_visual == True and 'mesh' in geometry}">
-        <xacro:property name="mesh_xyz" value="${geometry['mesh']['xyz']}" />
-        <xacro:property name="mesh_rpy" value="${geometry['mesh']['rpy']}" />
-        <xacro:property name="mesh_scale" value="${geometry['mesh']['scale']}" />
-        <xacro:property name="mesh_filename" value="${geometry['mesh']['filename']}" />
+          <xacro:property name="mesh_xyz"
+            value="${geometry['mesh']['xyz']}" />
+          <xacro:property name="mesh_rpy"
+            value="${geometry['mesh']['rpy']}" />
+          <xacro:property name="mesh_scale"
+            value="${geometry['mesh']['scale']}" />
+          <xacro:property name="mesh_filename"
+            value="${geometry['mesh']['filename']}" />
         </xacro:if>
         <!-- Camera Center -->
@@ -96,79 +114,14 @@
         </joint>
         <link name="${right_camera_optical_frame_name}"/>
-        <gazebo reference="${link_name}">
-          <material>Gazebo/DarkYellow </material>
-          <sensor type="multicamera" name="${prefix}${name}">
-            <update_rate>${frame_rate}</update_rate>
-            <camera name="left">
-              <pose>0 ${baseline/2} 0 0 0 0</pose>
-              <horizontal_fov>${horizontal_fov}</horizontal_fov>
-              <image>
-                <width>${image_width} </width>
-                <height>${image_height}</height>
-                <format>R8G8B8</format>
-              </image>
-              <clip>
-                <near>0.01</near>
-                <far>100</far>
-              </clip>
-              <!-- <noise>
-                <type>gaussian</type>
-                <mean>0.0</mean>
-                <stddev>0.007</stddev>
-              </noise>
-              <distortion>
-                <k1>0.0</k1>
-                <k2>0.0</k2>
-                <k3>0.0</k3>
-                <p1>0.0</p1>
-                <p2>0.0</p2>
-                <center>0.5 0.5</center>
-              </distortion> -->
-            </camera>
-            <camera name="right">
-              <pose>0 ${baseline/2} 0 0 0 0</pose>
-              <horizontal_fov>${horizontal_fov}</horizontal_fov>
-              <image>
-                <width>${image_width} </width>
-                <height>${image_height}</height>
-                <format>R8G8B8</format>
-              </image>
-              <clip>
-                <near>0.01</near>
-                <far>100</far>
-              </clip>
-              <!-- <noise>
-                <type>gaussian</type>
-                <mean>0.0</mean>
-                <stddev>0.007</stddev>
-              </noise>
-              <distortion>
-                <k1>0.0</k1>
-                <k2>0.0</k2>
-                <k3>0.0</k3>
-                <p1>0.0</p1>
-                <p2>0.0</p2>
-                <center>0.5 0.5</center>
-              </distortion> -->
-            </camera>
-            <plugin name="driver" filename="libgazebo_ros_camera.so">
-                <ros>
-                  <namespace>${ros_namespace}</namespace>
-                  <remapping>camera/left/image_raw:=left/image_raw</remapping>
-                  <remapping>camera/right/image_raw:=right/image_raw</remapping>
-                  <remapping>camera/left/camera_info:=left/camera_info</remapping>
-                  <remapping>camera/right/camera_info:=right/camera_info</remapping>
-                  <remapping>camera/left/image_raw/compressed:=left/image_raw/compressed</remapping>
-                  <remapping>camera/right/image_raw/compressed:=right/image_raw/compressed</remapping>
-                  <remapping>camera/left/image_raw/compressedDepth:=left/image_raw/compressedDepth</remapping>
-                  <remapping>camera/right/image_raw/compressedDepth:=right/image_raw/compressedDepth</remapping>
-                  <remapping>camera/left/image_raw/theora:=left/image_raw/theora</remapping>
-                  <remapping>camera/right/image_raw/theora:=right/image_raw/theora</remapping>
-                </ros>
-                <camera_name>camera</camera_name>
-                <frame_name>${link_name}</frame_name>
-            </plugin>
-          </sensor>
-        </gazebo>
+        <xacro:if value="${'simulation' in mode}">
+          <xacro:include filename="$(find romea_stereo_camera_description)/urdf/stereo_camera.simulation.xacro" />
+            <xacro:camera_stereo_sensor_simulation
+              prefix="${prefix}"
+              mode="${mode}"
+              name="${name}"
+              link_name="${link_name}"
+              configuration="${configuration}"
+              ros_namespace="${ros_namespace}"/>
+        </xacro:if>
     </xacro:macro>
 </robot>

Commit message: remove collision in URDF

File: romea_stereo_camera_description/urdf/stereo_camera.xacro (robot description, xacro)
@@ -81,10 +81,10 @@
                 </xacro:if>
             </visual>
-            <collision>
+            <!-- <collision>
                 <origin xyz="${aabb_center[0]} ${aabb_center[1]} ${aabb_center[2]}" rpy="0 0 0" />
                 <geometry>
                 <box size="${aabb_length} ${aabb_width} ${aabb_height}" />
                 </geometry>
-            </collision>
+            </collision> -->
         </link>
         <!-- Left Camera -->
